Commit message: feat: 🎸 new kuavo urdf to xml

File: loco_mujoco/environments/data/kuavo/kuavo.urdf (robot description, URDF)
Before this commit: robot biped_v2, 20 links, 19 joints
Links:
- removed link l_foot
- removed link l_larm
- removed link l_lleg
- removed link l_uarm
- removed link l_uarm_y
- removed link l_uarm_z
- removed link l_uleg
- removed link l_uleg_x
- removed link l_uleg_z
- removed link r_foot
- removed link r_larm
- removed link r_lleg
- removed link r_uarm
- removed link r_uarm_y
- removed link r_uarm_z
- removed link r_uleg
- removed link r_uleg_x
- removed link r_uleg_z
- removed link torso
- removed link world
- added link base_link, mass 7.71324827879796; collision mesh filename=./meshes/base_link.STL; visual mesh filename=./meshes/base_link.STL
- added link l_arm_pitch, mass 0.0855565384250596; collision mesh filename=./meshes/l_arm_pitch.STL; visual mesh filename=./meshes/l_arm_pitch.STL
- added link l_arm_roll, mass 0.243859089022774; collision mesh filename=./meshes/l_arm_roll.STL; visual mesh filename=./meshes/l_arm_roll.STL
- added link l_arm_yaw, mass 0.231645925727573; collision mesh filename=./meshes/l_arm_yaw.STL; visual mesh filename=./meshes/l_arm_yaw.STL
- added link l_foot_pitch, mass 0.00898868764931505; collision mesh filename=./meshes/l_foot_pitch.STL; visual mesh filename=./meshes/l_foot_pitch.STL
- added link l_foot_roll, mass 0.48595336841054; collision mesh filename=./meshes/l_foot_roll.STL; visual mesh filename=./meshes/l_foot_roll.STL
- added link l_forearm_pitch, mass 0.100717925891199; collision mesh filename=./meshes/l_forearm_pitch.STL; visual mesh filename=./meshes/l_forearm_pitch.STL
- added link l_forearm_yaw, mass 0.156174407901059; collision mesh filename=./meshes/l_forearm_yaw.STL; visual mesh filename=./meshes/l_forearm_yaw.STL
- added link l_hand_pitch, mass 0.0531311255846087; collision mesh filename=./meshes/l_hand_pitch.STL; visual mesh filename=./meshes/l_hand_pitch.STL
- added link l_hand_roll, mass 0.00225080087545489; collision mesh filename=./meshes/l_hand_roll.STL; visual mesh filename=./meshes/l_hand_roll.STL
- added link l_knee, mass 0.817175320465059; collision mesh filename=./meshes/l_knee.STL; visual mesh filename=./meshes/l_knee.STL
- added link l_l_arm_bar, mass 0.000933425350872019; collision mesh filename=./meshes/l_l_arm_bar.STL; visual mesh filename=./meshes/l_l_arm_bar.STL
- added link l_l_arm_tendon, mass 0.00374681809424582; collision mesh filename=./meshes/l_l_arm_tendon.STL; visual mesh filename=./meshes/l_l_arm_tendon.STL
- added link l_l_bar, mass 0.00874829869457794; collision mesh filename=./meshes/l_l_bar.STL; visual mesh filename=./meshes/l_l_bar.STL
- added link l_l_tendon, mass 0.083522124317674; collision mesh filename=./meshes/l_l_tendon.STL; visual mesh filename=./meshes/l_l_tendon.STL
- added link l_leg_pitch, mass 0.45065011418642; collision mesh filename=./meshes/l_leg_pitch.STL; visual mesh filename=./meshes/l_leg_pitch.STL
- added link l_leg_roll, mass 0.118529537524385; collision mesh filename=./meshes/l_leg_roll.STL; visual mesh filename=./meshes/l_leg_roll.STL
- added link l_leg_yaw, mass 0.20405278020544; collision mesh filename=./meshes/l_leg_yaw.STL; visual mesh filename=./meshes/l_leg_yaw.STL
- added link l_r_arm_bar, mass 0.00093342533722621; collision mesh filename=./meshes/l_r_arm_bar.STL; visual mesh filename=./meshes/l_r_arm_bar.STL
- added link l_r_arm_tendon, mass 0.00269247094438198; collision mesh filename=./meshes/l_r_arm_tendon.STL; visual mesh filename=./meshes/l_r_arm_tendon.STL
- added link l_r_bar, mass 0.00874829655091912; collision mesh filename=./meshes/l_r_bar.STL; visual mesh filename=./meshes/l_r_bar.STL
- added link l_r_tendon, mass 0.0780668768936421; collision mesh filename=./meshes/l_r_tendon.STL; visual mesh filename=./meshes/l_r_tendon.STL
- added link r_arm_pitch, mass 0.0855564935505709; collision mesh filename=./meshes/r_arm_pitch.STL; visual mesh filename=./meshes/r_arm_pitch.STL
- added link r_arm_roll, mass 0.24385908133804; collision mesh filename=./meshes/r_arm_roll.STL; visual mesh filename=./meshes/r_arm_roll.STL
- added link r_arm_yaw, mass 0.231645950350007; collision mesh filename=./meshes/r_arm_yaw.STL; visual mesh filename=./meshes/r_arm_yaw.STL
- added link r_foot_pitch, mass 0.00898868764931501; collision mesh filename=./meshes/r_foot_pitch.STL; visual mesh filename=./meshes/r_foot_pitch.STL
- added link r_foot_roll, mass 0.235882377040623; collision mesh filename=./meshes/r_foot_roll.STL; visual mesh filename=./meshes/r_foot_roll.STL
- added link r_forearm_pitch, mass 0.082246913288193; collision mesh filename=./meshes/r_forearm_pitch.STL; visual mesh filename=./meshes/r_forearm_pitch.STL
- added link r_forearm_yaw, mass 0.156174142689454; collision mesh filename=./meshes/r_forearm_yaw.STL; visual mesh filename=./meshes/r_forearm_yaw.STL
- added link r_hand_pitch, mass 0.0535643416316945; collision mesh filename=./meshes/r_hand_pitch.STL; visual mesh filename=./meshes/r_hand_pitch.STL
- added link r_hand_roll, mass 0.00225080086305129; collision mesh filename=./meshes/r_hand_roll.STL; visual mesh filename=./meshes/r_hand_roll.STL
- added link r_knee, mass 0.345443991337626; collision mesh filename=./meshes/r_knee.STL; visual mesh filename=./meshes/r_knee.STL
- added link r_l_arm_bar, mass 0.000933425428650283; collision mesh filename=./meshes/r_l_arm_bar.STL; visual mesh filename=./meshes/r_l_arm_bar.STL
- added link r_l_arm_tendon, mass 0.0026624084343365; collision mesh filename=./meshes/r_l_arm_tendon.STL; visual mesh filename=./meshes/r_l_arm_tendon.STL
- added link r_l_bar, mass 0.00874829521108898; collision mesh filename=./meshes/r_l_bar.STL; visual mesh filename=./meshes/r_l_bar.STL
- added link r_l_tendon, mass 0.0483474436719092; collision mesh filename=./meshes/r_l_tendon.STL; visual mesh filename=./meshes/r_l_tendon.STL
- added link r_leg_pitch, mass 0.448539615819603; collision mesh filename=./meshes/r_leg_pitch.STL; visual mesh filename=./meshes/r_leg_pitch.STL
- added link r_leg_roll, mass 0.11853067519234; collision mesh filename=./meshes/r_leg_roll.STL; visual mesh filename=./meshes/r_leg_roll.STL
- added link r_leg_yaw, mass 0.204051628397563; collision mesh filename=./meshes/r_leg_yaw.STL; visual mesh filename=./meshes/r_leg_yaw.STL
- added link r_r_arm_bar, mass 0.000933425431007405; collision mesh filename=./meshes/r_r_arm_bar.STL; visual mesh filename=./meshes/r_r_arm_bar.STL
- added link r_r_arm_tendon, mass 0.00373178797597326; collision mesh filename=./meshes/r_r_arm_tendon.STL; visual mesh filename=./meshes/r_r_arm_tendon.STL
- added link r_r_bar, mass 0.00874829774758129; collision mesh filename=./meshes/r_r_bar.STL; visual mesh filename=./meshes/r_r_bar.STL
- added link r_r_tendon, mass 0.053802691494778; collision mesh filename=./meshes/r_r_tendon.STL; visual mesh filename=./meshes/r_r_tendon.STL
- added link real_camera_link, mass 0.0173287679990781; collision mesh filename=./meshes/real_camera_link.STL; visual mesh filename=./meshes/real_camera_link.STL
Joints:
- removed joint l_ankle
- removed joint l_elbow
- removed joint l_hip_x
- removed joint l_hip_y
- removed joint l_hip_z
- removed joint l_shoulder_x
- removed joint l_shoulder_y
- removed joint l_shoulder_z
- removed joint r_ankle
- removed joint r_elbow
- removed joint r_hip_x
- removed joint r_hip_y
- removed joint r_hip_z
- removed joint r_shoulder_x
- removed joint r_shoulder_y
- removed joint r_shoulder_z
- removed joint world_joint
- added joint camera_joint: type fixed, parent base_link, child real_camera_link, origin xyz=0.078507 0.0026635 0.47328 rpy=0 0.61087 0, axis 0 0 0
- added joint l_arm_pitch: type continuous, parent base_link, child l_arm_pitch, origin xyz=-0.0174998525199999 0.121 0.3145 rpy=0 0 0, axis 0 1 0
- added joint l_arm_roll: type continuous, parent l_arm_pitch, child l_arm_roll, origin xyz=0.0638750000000005 0.143475 0 rpy=0 0 0, axis -1 0 0
- added joint l_arm_yaw: type continuous, parent l_arm_roll, child l_arm_yaw, origin xyz=-0.0436732904500001 -0.000228544867618807 -0.0507499999999994 rpy=0 0 0, axis 0 0.0045033014816499 0.999989860086474
- added joint l_foot_pitch: type continuous, parent l_knee, child l_foot_pitch, origin xyz=9.39839333040909E-05 0.0209999999999999 -0.346142421968556 rpy=0 0 0, axis 0 -1 0
- added joint l_foot_roll: type continuous, parent l_foot_pitch, child l_foot_roll, origin xyz=0.021 -0.021 0.000142421968555073 rpy=0 0 0, axis -1 0 0
- added joint l_forearm_pitch: type continuous, parent l_arm_yaw, child l_forearm_pitch, origin xyz=0 -0.0300214551323814 -0.1357 rpy=0 0 0, axis 0 1 0
- added joint l_forearm_yaw: type continuous, parent l_forearm_pitch, child l_forearm_yaw, origin xyz=0 0.0302500000000002 -0.0915499999999999 rpy=0 0 0, axis 0 0 -1
- added joint l_hand_pitch: type continuous, parent l_hand_roll, child l_hand_pitch, origin xyz=0.02137 0 0 rpy=0 0 0, axis -1 0 0
- added joint l_hand_roll: type continuous, parent l_forearm_yaw, child l_hand_roll, origin xyz=-0.025322 0 -0.1575 rpy=0 0 0, axis -1 0 0
- added joint l_l_arm_bar: type continuous, parent l_forearm_yaw, child l_l_arm_bar, origin xyz=0.011299999998424 0.024140000000002 -0.0759999999999971 rpy=0 0 0, axis 0 -1 0
- added joint l_l_arm_tendon: type continuous, parent l_l_arm_bar, child l_l_arm_tendon, origin xyz=-0.0159983282022835 0.0040000013363603 0.000231289282113974 rpy=0 0 0, axis 0 1 0
- added joint l_l_bar: type continuous, parent l_knee, child l_l_bar, origin xyz=9.39839333040753E-05 0.0294999999999999 -0.090000000000001 rpy=0 0 0, axis 0 -1 0
- added joint l_l_tendon: type continuous, parent l_l_bar, child l_l_tendon, origin xyz=-0.0576888204074241 -0.00450000000000017 0.00599999999999978 rpy=0 0 0, axis 0 1 0
- added joint l_leg_pitch: type continuous, parent l_leg_yaw, child l_leg_pitch, origin xyz=0 0.0939999999999999 -0.13645 rpy=0 0 0, axis 0 -1 0
- added joint l_leg_roll: type continuous, parent base_link, child l_leg_roll, origin xyz=-0.0756149468145449 0.087 -0.0720754569616772 rpy=0 0 0, axis -1 0 0
- added joint l_leg_yaw: type continuous, parent l_leg_roll, child l_leg_yaw, origin xyz=0.0735 0 0.0130000000000001 rpy=0 0 0, axis 0 0 1
- added joint l_r_arm_bar: type continuous, parent l_forearm_yaw, child l_r_arm_bar, origin xyz=0.011300000004892 -0.024139999999997 -0.1145 rpy=0 0 0, axis 0 1 0
- added joint l_r_arm_tendon: type continuous, parent l_r_arm_bar, child l_r_arm_tendon, origin xyz=-0.0159983310229197 -0.00400002806712421 0.000231094095741222 rpy=0 0 0, axis 0 -1 0
- added joint l_r_bar: type continuous, parent l_knee, child l_r_bar, origin xyz=9.39839333042539E-05 -0.0295 -0.153000000000001 rpy=0 0 0, axis 0 1 0
- added joint l_r_tendon: type continuous, parent l_r_bar, child l_r_tendon, origin xyz=-0.0576888204074239 0.00508602348130947 0.00600000000000012 rpy=0 0 0, axis 0 -1 0
- added joint r_arm_pitch: type continuous, parent base_link, child r_arm_pitch, origin xyz=-0.0174998525199999 -0.126 0.3145 rpy=0 0 0, axis 0 -1 0
- added joint r_arm_roll: type continuous, parent r_arm_pitch, child r_arm_roll, origin xyz=0.0638750000000006 -0.138475 0 rpy=0 0 0, axis -1 0 0
- added joint r_arm_yaw: type continuous, parent r_arm_roll, child r_arm_yaw, origin xyz=-0.0436749999999998 0 -0.0497499999999998 rpy=0 0 0, axis 0 0 -1
- added joint r_foot_pitch: type continuous, parent r_knee, child r_foot_pitch, origin xyz=0 -0.021 -0.346000000000001 rpy=0 0 0, axis 0 -1 0
- added joint r_foot_roll: type continuous, parent r_foot_pitch, child r_foot_roll, origin xyz=0.021 0.0209999999999999 0 rpy=0 0 0, axis -1 0 0
- added joint r_forearm_pitch: type continuous, parent r_arm_yaw, child r_forearm_pitch, origin xyz=0 0.0302500000000003 -0.1377 rpy=0 0 0, axis 0 -1 0
- added joint r_forearm_yaw: type continuous, parent r_forearm_pitch, child r_forearm_yaw, origin xyz=0 -0.0302500000000002 -0.0905499999999999 rpy=0 0 0, axis 0 0 1
- added joint r_hand_pitch: type continuous, parent r_hand_roll, child r_hand_pitch, origin xyz=0.02137 0 0 rpy=0 0 0, axis 0 1 0
- added joint r_hand_roll: type continuous, parent r_forearm_yaw, child r_hand_roll, origin xyz=-0.025322 0 -0.1575 rpy=0 0 0, axis -1 0 0
- added joint r_l_arm_bar: type continuous, parent r_forearm_yaw, child r_l_arm_bar, origin xyz=0.0113000000048921 0.024139999999997 -0.1145 rpy=0 0 0, axis 0 -1 0
- added joint r_l_arm_tendon: type continuous, parent r_l_arm_bar, child r_l_arm_tendon, origin xyz=-0.0159983310229197 0.00400002806712421 0.000231094095741222 rpy=0 0 0, axis 0 -1 0
- added joint r_l_bar: type continuous, parent r_knee, child r_l_bar, origin xyz=0 0.0294999999999999 -0.153000000000001 rpy=0 0 0, axis 0 -1 0
- added joint r_l_tendon: type continuous, parent r_l_bar, child r_l_tendon, origin xyz=-0.0576888204074239 -0.00449999999999988 0.00600000000000001 rpy=0 0 0, axis 0 1 0
- added joint r_leg_pitch: type continuous, parent r_leg_yaw, child r_leg_pitch, origin xyz=0 -0.094 -0.13645 rpy=0 0 0, axis 0 -1 0
- added joint r_leg_roll: type continuous, parent base_link, child r_leg_roll, origin xyz=-0.0756149468145449 -0.087 -0.0720754569616772 rpy=0 0 0, axis -1 0 0
- added joint r_leg_yaw: type continuous, parent r_leg_roll, child r_leg_yaw, origin xyz=0.0735 0 0.0130000000000001 rpy=0 0 0, axis 0 0 1
- added joint r_r_arm_bar: type continuous, parent r_forearm_yaw, child r_r_arm_bar, origin xyz=0.0112999999984239 -0.024140000000002 -0.0759999999999971 rpy=0 0 0, axis 0 1 0
- added joint r_r_arm_tendon: type continuous, parent r_r_arm_bar, child r_r_arm_tendon, origin xyz=-0.0159983282022835 -0.0040000013363603 0.000231289282113974 rpy=0 0 0, axis 0 1 0
- added joint r_r_bar: type continuous, parent r_knee, child r_r_bar, origin xyz=0 -0.0294999999999999 -0.0900000000000002 rpy=0 0 0, axis 0 -1 0
- added joint r_r_tendon: type continuous, parent r_r_bar, child r_r_tendon, origin xyz=-0.0576888204074261 0.00450000000000034 0.00599999999999878 rpy=0 0 0, axis 0 1 0
- joint l_knee: child l_lleg -> l_knee; limit lower=-0.174 upper=2.53 effort=74 velocity=47 -> (none); origin xyz=0 0.03365 -0.23 rpy=0 0 0 -> xyz=0.00413596009601052 -0.0686389599620252 -0.249965785326798 rpy=0 0 0; parent l_uleg -> l_leg_pitch; type revolute -> continuous
- joint r_knee: axis 0 1 0 -> 0 -1 0; child r_lleg -> r_knee; limit lower=-0.174 upper=2.53 effort=74 velocity=47 -> (none); origin xyz=0 -0.03365 -0.23 rpy=0 0 0 -> xyz=0.00413596009601069 0.0685500000000013 -0.249965785326798 rpy=0 0 0; parent r_uleg -> r_leg_pitch; type revolute -> continuous
